File: Development_Board_ESP32-V1.0/Development_Board_ESP32-V1.0.kicad_pcb (KiCad board)
At the start: 2 copper layers, 100 x 100 mm, 148 parts, among them J1 USB_B, J2 GPIO, J3 OLED, Q1 MMBT3904, Q2 MMBT3904, Q3 MMBT3904, Q4 MMBT3904, Q5 MMBT3904, Q6 MMBT3904, U1 ESP32-WROOM-32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

Commit message: Subiendo todo por si cambio
Parts:
- R5: value 1K -> 470
Changed lines of the file:
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@@
 			(psa4output no)
 			(plot_black_and_white yes)
-			(plotinvisibletext no)
 			(sketchpadsonfab no)
 			(plotpadnumbers no)
@@
 			)
 		)
-		(property "Value" "1K"
+		(property "Value" "470"
 			(at 0 1.82 0)
 			(layer "F.Fab")
@@
 	)
 	(zone
-		(net 68)
-		(net_name "IO2{slash}LED")
-		(layer "F.Cu")
-		(name "$teardrop_padvia$")
-		(hatch full 0.1)
-		(priority 30102)
-		(attr
-			(teardrop
-				(type padvia)
-			)
-		)
-		(connect_pads yes
-			(clearance 0)
-		)
-		(min_thickness 0.0254)
-		(filled_areas_thickness no)
-		(fill yes
-			(thermal_gap 0.5)
-			(thermal_bridge_width 0.5)
-			(island_removal_mode 1)
-			(island_area_min 10)
-		)
-		(polygon
-			(pts
-				(xy 63.302 110.5154) (xy 63.302 110.2614) (xy 62.649521 109.725537) (xy 62.001 110.363) (xy 62.644503 111.025687)
-			)
-		)
-	)
-	(zone
 		(net 8)
 		(net_name "+3.3V")
@@
 	)
 	(zone
-		(net 15)
-		(net_name "Net-(D3-A)")
-		(layer "F.Cu")
-		(name "$teardrop_padvia$")
-		(hatch full 0.1)
-		(priority 30106)
-		(attr
-			(teardrop
-				(type padvia)
-			)
-		)
-		(connect_pads yes
-			(clearance 0)
-		)
-		(min_thickness 0.0254)
-		(filled_areas_thickness no)
-		(fill yes
-			(thermal_gap 0.5)
-			(thermal_bridge_width 0.5)
-			(island_removal_mode 1)
-			(island_area_min 10)
-		)
-		(polygon
-			(pts
-				(xy 57.602 110.236) (xy 57.602 110.49) (xy 58.256973 111.013) (xy 58.903 110.363) (xy 58.256973 109.713)
-			)
-		)
-	)
-	(zone
 		(net 11)
 		(net_name "RX")
@@
 	)
 	(zone
+		(net 15)
+		(net_name "Net-(D3-A)")
+		(layer "F.Cu")
+		(name "$teardrop_padvia$")
+		(hatch full 0.1)
+		(priority 30001)
+		(attr
+			(teardrop
+				(type padvia)
+			)
+		)
+		(connect_pads yes
+			(clearance 0)
+		)
+		(min_thickness 0.0254)
+		(filled_areas_thickness no)
+		(fill yes
+			(thermal_gap 0.5)
+			(thermal_bridge_width 0.5)
+			(island_removal_mode 1)
+			(island_area_min 10)
+		)
+		(polygon
+			(pts
+				(xy 57.602 110.236) (xy 57.602 110.49) (xy 58.256973 111.013) (xy 58.903 110.363) (xy 58.256973 109.713)
+			)
+		)
+	)
+	(zone
 		(net 1)
 		(net_name "+5V")
@@
 			)
 		)
+	)
+	(zone
+		(net 68)
+		(net_name "IO2{slash}LED")
+		(layer "F.Cu")
+		(name "$teardrop_padvia$")
+		(hatch full 0.1)
+		(priority 30000)
+		(attr
+			(teardrop
+				(type padvia)
+			)
+		)
+		(connect_pads yes
+			(clearance 0)
+		)
+		(min_thickness 0.0254)
+		(filled_areas_thickness no)
+		(fill yes
+			(thermal_gap 0.5)
+			(thermal_bridge_width 0.5)
+			(island_removal_mode 1)
+			(island_area_min 10)
+		)
+		(polygon
+			(pts
+				(xy 63.302 110.5154) (xy 63.302 110.2614) (xy 62.649521 109.725537) (xy 62.001 110.363) (xy 62.644503 111.025687)
+			)
+		)
